File: pcb/sd.kicad_sch (KiCad schematic)
At the start: 2 parts, among them J5 Micro_SD_Card_Det_Hirose_DM3AT

Commit message: Merging in work from FSAE repo from when I forgot this one existed
Parts:
- gave numbers to parts that had none: 1
Connections:
- net SD_DATA1: no longer names the net of J5.8 (DAT1)
- net SD_DATA2: no longer names the net of J5.1 (DAT2)
- net SD_DATA3: no longer names the net of J5.2 (DAT3/CD)
- no-connect marks 0 -> 3
Changed lines of the file:
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@@
 		(color 0 0 0 0)
 	)
+	(no_connect
+		(at 129.54 83.82)
+	)
+	(no_connect
+		(at 129.54 86.36)
+	)
+	(no_connect
+		(at 129.54 101.6)
+	)
 	(wire
 		(pts
@@
 	(wire
 		(pts
-			(xy 123.19 86.36) (xy 129.54 86.36)
-		)
-		(stroke
-			(width 0)
-			(type default)
-		)
-	)
-	(wire
-		(pts
 			(xy 173.99 106.68) (xy 173.99 109.22)
 		)
@@
 	(wire
 		(pts
-			(xy 123.19 83.82) (xy 129.54 83.82)
-		)
-		(stroke
-			(width 0)
-			(type default)
-		)
-	)
-	(wire
-		(pts
 			(xy 123.19 93.98) (xy 129.54 93.98)
 		)
@@
 		(pts
 			(xy 129.54 91.44) (xy 102.87 91.44)
-		)
-		(stroke
-			(width 0)
-			(type default)
-		)
-	)
-	(wire
-		(pts
-			(xy 123.19 101.6) (xy 129.54 101.6)
 		)
 		(stroke
@@
 		(shape input)
 		(at 123.19 88.9 180)
-		(effects
-			(font
-				(size 1.27 1.27)
-			)
-			(justify right)
-		)
-	)
-	(hierarchical_label "SD_DATA1"
-		(shape bidirectional)
-		(at 123.19 101.6 180)
-		(effects
-			(font
-				(size 1.27 1.27)
-			)
-			(justify right)
-		)
-	)
-	(hierarchical_label "SD_DATA3"
-		(shape bidirectional)
-		(at 123.19 86.36 180)
-		(effects
-			(font
-				(size 1.27 1.27)
-			)
-			(justify right)
-		)
-	)
-	(hierarchical_label "SD_DATA2"
-		(shape bidirectional)
-		(at 123.19 83.82 180)
 		(effects
 			(font
@@
 		(dnp no)
 		(fields_autoplaced yes)
-		(property "Reference" "C?"
+		(property "Reference" "C4"
 			(at 90.17 92.7099 0)
 			(effects
@@
 			(project ""
 				(path "/1f94b0a1-b989-49dc-a3ab-12a0e728079d/a157da69-e8fe-4b49-9cb0-61544ea7d730"
-					(reference "C?")
+					(reference "C4")
 					(unit 1)
 				)
