File: pcb/circuit_protection.kicad_sch (KiCad schematic)
At the start: 26 parts, among them U1 TPS259474ARPWR

Commit message: Merging in work from FSAE repo from when I forgot this one existed
Parts:
- removed C4, C5, C6, C7: C, symbol Device:C
- removed D6: LED, symbol Device:LED
- removed R20, R21, R22, R23, R24, R25, R26: R, symbol Device:R
- removed U1, U?: TPS259474ARPWR, TPS259474ARPWR:IC_TPS259474ARPWR, symbol ev24:TPS259474ARPWR
- added JP1: SolderJumper_2_Open, Jumper:SolderJumper-2_P1.3mm_Open_RoundedPad1.0x1.5mm, symbol Jumper:SolderJumper_2_Open
- added U1: TPS259474ARPWR, 0_tps259474arpwr:IC_TPS259474ARPWR, symbol 0_tps259474arpwr:TPS259474ARPWR
- C1: footprint (none) -> Capacitor_SMD:C_0402_1005Metric
- C2: value C -> 1.2n; footprint (none) -> Capacitor_SMD:C_0402_1005Metric
- C3: value C -> 3300p; footprint (none) -> Capacitor_SMD:C_0402_1005Metric
- C5: renamed from C?; value C -> 1u; footprint (none) -> Capacitor_SMD:C_0402_1005Metric
- D8: renamed from D?; footprint (none) -> Diode_SMD:D_0402_1005Metric
- R1: value R -> 18k; footprint (none) -> Resistor_SMD:R_0402_1005Metric
- R16: value R -> 1.6k; footprint (none) -> Resistor_SMD:R_0402_1005Metric
- R17: value R -> ~; footprint (none) -> Resistor_SMD:R_0402_1005Metric
- R18: footprint (none) -> Resistor_SMD:R_0402_1005Metric
- R19: value R -> 500; footprint (none) -> Resistor_SMD:R_0402_1005Metric
- R2: value R -> 55k; footprint (none) -> Resistor_SMD:R_0402_1005Metric
- R20: renamed from R?; value R -> 91k; footprint (none) -> Resistor_SMD:R_0402_1005Metric
Connections:
- net +3v3: now also JP1.2 (B), U1.6 (OUT)
- net +3v3_UNFUSED: now also JP1.1 (A), U1.5 (IN)
- net GND: now also U1.8 (GND)
- net at R16.1: now also U1.9 (ILM)
- net at R1.1, R20.2: now also U1.1 (EN/UVLO)
- net at C2.1: now also U1.10 (ITIMER)
- net at R1.2, R2.1: now also U1.2 (OVLO)
- net at R17.2, R18.1: now also U1.4 (PGTH)
- net at C3.1: now also U1.7 (DVDT)
- no-connect marks 0 -> 1
Other:
- note added: "Power Good is just a depletion nmos that is connected to ground, see page 24 of datasheet This results in a leakage current of 6.6mA at 3.3V when not good, but I don't really care about that"
- note removed: "Look up how the PG pin works in more detail"
- moved on the sheet: C2, C3, C5, D8, R1, R16, R2, R20

Commit message: Quite a few changes
Other:
- note added: "Emergency power jumper for when I immediately realize I fucked something up"
Changed lines of the file:
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@@
+		)
+	)
+	(text "Emergency power jumper for when I \nimmediately realize I fucked something up"
+		(exclude_from_sim no)
+		(at 86.868 26.416 0)
+		(effects
+			(font
+				(size 1.27 1.27)
+			)
 		)
 	)
@@
 	)
 	(junction
+		(at 55.88 38.1)
+		(diameter 0)
+		(color 0 0 0 0)
+	)
+	(junction
 		(at 53.34 85.09)
 		(diameter 0)
@@
 	(junction
 		(at 123.19 38.1)
-		(diameter 0)
-		(color 0 0 0 0)
-	)
-	(junction
-		(at 60.96 38.1)
 		(diameter 0)
 		(color 0 0 0 0)
@@
 	(wire
 		(pts
-			(xy 60.96 22.86) (xy 82.55 22.86)
+			(xy 55.88 22.86) (xy 82.55 22.86)
 		)
 		(stroke
@@
 	(wire
 		(pts
-			(xy 60.96 38.1) (xy 66.04 38.1)
-		)
-		(stroke
-			(width 0)
-			(type default)
-		)
-	)
-	(wire
-		(pts
 			(xy 123.19 53.34) (xy 123.19 58.42)
 		)
@@
 	(wire
 		(pts
-			(xy 60.96 38.1) (xy 60.96 22.86)
-		)
-		(stroke
-			(width 0)
-			(type default)
-		)
-	)
-	(wire
-		(pts
-			(xy 53.34 38.1) (xy 60.96 38.1)
+			(xy 55.88 38.1) (xy 55.88 22.86)
+		)
+		(stroke
+			(width 0)
+			(type default)
+		)
+	)
+	(wire
+		(pts
+			(xy 53.34 38.1) (xy 55.88 38.1)
 		)
 		(stroke
@@
 		)
 		(stroke
+			(width 0)
+			(type default)
+		)
+	)
+	(wire
+		(pts
+			(xy 55.88 38.1) (xy 66.04 38.1)
+		)
+		(stroke
