File: pcb/driver-radio.kicad_sch (KiCad schematic)
At the start: 37 parts, among them J3 Conn_01x02_MountingPin, J4 Conn_01x02_MountingPin, J6 Conn_Coaxial

Commit message: Merging in work from FSAE repo from when I forgot this one existed
Parts:
- removed TP13: SD1, ev24-footprint-library:tp-ev24-nobacksilk, symbol Connector:TestPoint_Small
- removed TP14: SD2, ev24-footprint-library:tp-ev24-nobacksilk, symbol Connector:TestPoint_Small
- removed TP15: SD3, ev24-footprint-library:tp-ev24-nobacksilk, symbol Connector:TestPoint_Small
- added R21, R22, R23: 10k, Resistor_SMD:R_0402_1005Metric_Pad0.72x0.64mm_HandSolder, symbol Device:R
- D3, D5: footprint (none) -> LED_SMD:LED_0402_1005Metric
- D4: footprint (none) -> LED_SMD:LED_0402_1005Metric; now fitted; now in the parts list
- D6: renamed from D?; footprint (none) -> LED_SMD:LED_0402_1005Metric; now fitted; now in the parts list
- R11, R13: now fitted; now in the parts list
- TP1, TP10, TP12, TP16, TP2, TP3, TP4, TP5, TP6, TP7, TP8, TP9: footprint ev24-footprint-library:tp-ev24-nobacksilk -> 0_tp-ev24-nobacksilk:tp-ev24-nobacksilk
- TP11, TP17: footprint TestPoint:TestPoint_Pad_1.0x1.0mm -> 0_tp-ev24-nobacksilk:tp-ev24-nobacksilk
Connections:
- net +5V_UNFUSED is gone; now on net +5V: H4.1
- net +3V3: now also R21.2, R22.2, R23.2
- net MCU/CAR_HEARTBEAT: now also R12.1; no longer R10.1
- net MCU/SD_CLK: now also R23.1
- net MCU/SD_CMD: now also R22.1
- net MCU/SD_DATA0: now also R21.1
- net MCU/WARNING: now also R10.1; no longer R12.1
- net MCU/MAIN_LOOP: now reaches R11.1
- net MCU/FAULT: now reaches R13.1
- no-connect marks 2 -> 0
Other:
- sheet Circuit Protection ports: added none; removed +5v, +5v_UNFUSED
- sheet MCU ports: added FAULT, MAIN_LOOP, RADIO ON/OFF; removed SD_DATA1, SD_DATA2, SD_DATA3
- sheet SD Card Adaptor ports: added none; removed SD_DATA1, SD_DATA2, SD_DATA3
- note removed: "Not including all these LEDs so I can go full speed on SD card"
- moved on the sheet: D3, D5, R10, R12

Commit message: Quite a few changes
Parts:
- D3: value LED -> BLU; IPN (none) -> DIO-000160-00
- D4: value LED -> GRN; IPN (none) -> LED-000534-00
- D5: value LED -> YLW; IPN (none) -> DIO-000505-00
- D6: value LED -> RED; IPN (none) -> DIO-000152-00
Connections:
- net MCU/CAR_HEARTBEAT: now also R10.1; no longer R12.1
- net MCU/WARNING: now also R12.1; no longer R10.1
- net at R12.2: now also D5.2 (A); no longer D3.2 (A)
- net at R10.2: now also D3.2 (A); no longer D5.2 (A)
Other:
- sheet MCU ports: added ESP32_RF_RX, ESP32_RF_TX, IS_RADIO_RECIEVING; removed RADIO_STATUS, RF_RX, RF_TX
- moved on the sheet: R10, R12
Changed lines of the file:
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@@
 	(symbol
 		(lib_id "Device:R_Small_US")
-		(at 81.28 97.79 270)
+		(at 81.28 73.66 270)
 		(unit 1)
 		(exclude_from_sim no)
@@
 		(dnp no)
 		(property "Reference" "R12"
-			(at 79.375 99.695 90)
+			(at 79.375 75.565 90)
 			(effects
 				(font
@@
 		)
 		(property "Value" "500"
-			(at 79.375 102.235 90)
+			(at 79.375 78.105 90)
 			(effects
 				(font
@@
 		)
 		(property "Footprint" "Resistor_SMD:R_0402_1005Metric"
-			(at 81.28 97.79 0)
+			(at 81.28 73.66 0)
 			(effects
 				(font
@@
 		)
 		(property "Datasheet" "~"
-			(at 81.28 97.79 0)
+			(at 81.28 73.66 0)
 			(effects
 				(font
@@
 		)
 		(property "Description" "Resistor, small US symbol"
-			(at 81.28 97.79 0)
+			(at 81.28 73.66 0)
 			(effects
 				(font
@@
 		)
 		(property "MANUFACTURER" ""
-			(at 81.28 97.79 0)
+			(at 81.28 73.66 0)
 			(effects
 				(font
@@
 		)
 		(property "MAXIMUM_PACKAGE_HEIGHT" ""
-			(at 81.28 97.79 0)
+			(at 81.28 73.66 0)
 			(effects
 				(font
@@
 		)
 		(property "PARTREV" ""
-			(at 81.28 97.79 0)
+			(at 81.28 73.66 0)
 			(effects
 				(font
@@
 		)
 		(property "STANDARD" ""
-			(at 81.28 97.79 0)
+			(at 81.28 73.66 0)
 			(effects
 				(font
@@
 		)
 		(property "SNAPEDA_PN" ""
-			(at 81.28 97.79 0)
+			(at 81.28 73.66 0)
 			(effects
 				(font
@@
 		)
 		(property "IPN" "RES-000545-00"
-			(at 81.28 97.79 0)
+			(at 81.28 73.66 0)
 			(effects
 				(font
@@
 			)
 		)
-		(property "Value" "LED"
+		(property "Value" "GRN"
 			(at 71.4375 92.0749 0)
 			(effects
@@
 			)
 		)
-		(property "Datasheet" "~"
+		(property "Datasheet" ""
 			(at 74.93 85.09 0)
 			(effects
@@
 			)
 		)
-		(property "Sim.Pins" "1=K 2=A"
+		(property "IPN" "LED-000534-00"
+			(at 74.93 85.09 0)
+			(effects
+				(font
+					(size 1.27 1.27)
+				)
+				(hide yes)
+			)
+		)
+		(property "MANUFACTURER" ""
+			(at 74.93 85.09 0)
+			(effects
+				(font
+					(size 1.27 1.27)
+				)
+				(hide yes)
+			)
+		)
+		(property "MAXIMUM_PACKAGE_HEIGHT" ""
+			(at 74.93 85.09 0)
+			(effects
+				(font
+					(size 1.27 1.27)
+				)
+				(hide yes)
+			)
+		)
+		(property "PARTREV" ""
+			(at 74.93 85.09 0)
+			(effects
+				(font
+					(size 1.27 1.27)
+				)
+				(hide yes)
+			)
+		)
+		(property "SNAPEDA_PN" ""
+			(at 74.93 85.09 0)
+			(effects
+				(font
+					(size 1.27 1.27)
+				)
+				(hide yes)
+			)
+		)
+		(property "STANDARD" ""
 			(at 74.93 85.09 0)
 			(effects
@@
 			)
 		)
-		(property "Value" "LED"
+		(property "Value" "YLW"
 			(at 71.4375 80.6449 0)
 			(effects
@@
 			)
 		)
-		(property "Datasheet" "~"
+		(property "Datasheet" ""
 			(at 74.93 73.66 0)
 			(effects
@@
 			)
 		)
-		(property "Sim.Pins" "1=K 2=A"
+		(property "IPN" "DIO-000505-00"
+			(at 74.93 73.66 0)
+			(effects
+				(font
+					(size 1.27 1.27)
+				)
+				(hide yes)
+			)
+		)
+		(property "MANUFACTURER" ""
+			(at 74.93 73.66 0)
+			(effects
+				(font
+					(size 1.27 1.27)
+				)
+				(hide yes)
+			)
+		)
+		(property "MAXIMUM_PACKAGE_HEIGHT" ""
+			(at 74.93 73.66 0)
+			(effects
+				(font
+					(size 1.27 1.27)
+				)
+				(hide yes)
+			)
+		)
+		(property "PARTREV" ""
+			(at 74.93 73.66 0)
+			(effects
+				(font
+					(size 1.27 1.27)
+				)
+				(hide yes)
+			)
+		)
+		(property "SNAPEDA_PN" ""
+			(at 74.93 73.66 0)
+			(effects
+				(font
+					(size 1.27 1.27)
+				)
+				(hide yes)
+			)
+		)
+		(property "STANDARD" ""
 			(at 74.93 73.66 0)
 			(effects
@@
 	(symbol
 		(lib_id "Device:R_Small_US")
-		(at 81.28 73.66 270)
+		(at 81.28 97.79 270)
 		(unit 1)
 		(exclude_from_sim no)
@@
 		(dnp no)
 		(property "Reference" "R10"
-			(at 79.375 75.565 90)
+			(at 79.375 99.695 90)
 			(effects
 				(font
@@
 		)
 		(property "Value" "500"
-			(at 79.375 78.105 90)
+			(at 79.375 102.235 90)
 			(effects
 				(font
@@
 		)
 		(property "Footprint" "Resistor_SMD:R_0402_1005Metric"
-			(at 81.28 73.66 0)
+			(at 81.28 97.79 0)
 			(effects
 				(font
@@
 		)
 		(property "Datasheet" "~"
-			(at 81.28 73.66 0)
+			(at 81.28 97.79 0)
 			(effects
 				(font
@@
 		)
 		(property "Description" "Resistor, small US symbol"
-			(at 81.28 73.66 0)
+			(at 81.28 97.79 0)
 			(effects
 				(font
@@
 		)
 		(property "MANUFACTURER" ""
-			(at 81.28 73.66 0)
+			(at 81.28 97.79 0)
 			(effects
 				(font
@@
 		)
 		(property "MAXIMUM_PACKAGE_HEIGHT" ""
-			(at 81.28 73.66 0)
+			(at 81.28 97.79 0)
 			(effects
 				(font
@@
 		)
 		(property "PARTREV" ""
-			(at 81.28 73.66 0)
+			(at 81.28 97.79 0)
 			(effects
 				(font
@@
 		)
 		(property "STANDARD" ""
-			(at 81.28 73.66 0)
+			(at 81.28 97.79 0)
 			(effects
 				(font
@@
 		)
 		(property "SNAPEDA_PN" ""
-			(at 81.28 73.66 0)
+			(at 81.28 97.79 0)
 			(effects
 				(font
@@
 		)
 		(property "IPN" "RES-000545-00"
-			(at 81.28 73.66 0)
+			(at 81.28 97.79 0)
 			(effects
 				(font
@@
 			)
 		)
-		(property "Value" "LED"
+		(property "Value" "BLU"
 			(at 71.4375 104.7749 0)
 			(effects
@@
 			)
 		)
-		(property "Datasheet" "~"
+		(property "Datasheet" ""
 			(at 74.93 97.79 0)
 			(effects
@@
 			)
 		)
-		(property "Sim.Pins" "1=K 2=A"
+		(property "IPN" "DIO-000160-00"
+			(at 74.93 97.79 0)
+			(effects
+				(font
+					(size 1.27 1.27)
+				)
+				(hide yes)
+			)
+		)
+		(property "MANUFACTURER" ""
+			(at 74.93 97.79 0)
+			(effects
+				(font
+					(size 1.27 1.27)
+				)
+				(hide yes)
+			)
+		)
+		(property "MAXIMUM_PACKAGE_HEIGHT" ""
+			(at 74.93 97.79 0)
+			(effects
+				(font
+					(size 1.27 1.27)
+				)
+				(hide yes)
+			)
+		)
+		(property "PARTREV" ""
+			(at 74.93 97.79 0)
+			(effects
+				(font
+					(size 1.27 1.27)
+				)
+				(hide yes)
+			)
+		)
+		(property "SNAPEDA_PN" ""
+			(at 74.93 97.79 0)
+			(effects
+				(font
+					(size 1.27 1.27)
+				)
+				(hide yes)
+			)
+		)
+		(property "STANDARD" ""
 			(at 74.93 97.79 0)
 			(effects
@@
 			)
 		)
-		(property "Value" "LED"
+		(property "Value" "RED"
 			(at 71.4375 116.2049 0)
 			(effects
@@
 			)
 		)
-		(property "Datasheet" "~"
+		(property "Datasheet" ""
 			(at 74.93 109.22 0)
 			(effects
@@
 			)
 		)
-		(property "Sim.Pins" "1=K 2=A"
+		(property "IPN" "DIO-000152-00"
+			(at 74.93 109.22 0)
+			(effects
+				(font
+					(size 1.27 1.27)
+				)
+				(hide yes)
+			)
+		)
+		(property "MANUFACTURER" ""
+			(at 74.93 109.22 0)
+			(effects
+				(font
+					(size 1.27 1.27)
+				)
+				(hide yes)
+			)
+		)
+		(property "MAXIMUM_PACKAGE_HEIGHT" ""
+			(at 74.93 109.22 0)
+			(effects
+				(font
+					(size 1.27 1.27)
+				)
+				(hide yes)
+			)
+		)
+		(property "PARTREV" ""
+			(at 74.93 109.22 0)
+			(effects
+				(font
+					(size 1.27 1.27)
+				)
+				(hide yes)
+			)
+		)
+		(property "SNAPEDA_PN" ""
+			(at 74.93 109.22 0)
+			(effects
+				(font
+					(size 1.27 1.27)
+				)
+				(hide yes)
+			)
+		)
+		(property "STANDARD" ""
 			(at 74.93 109.22 0)
 			(effects
@@
 			)
 		)
-		(pin "RF_TX" output
-			(at 137.16 53.34 0)
-			(effects
-				(font
-					(size 1.27 1.27)
-				)
-				(justify right)
-			)
-		)
-		(pin "RF_RX" input
-			(at 137.16 57.15 0)
-			(effects
-				(font
-					(size 1.27 1.27)
-				)
-				(justify right)
-			)
-		)
-		(pin "RADIO_STATUS" input
+		(pin "IS_RADIO_RECIEVING" input
 			(at 137.16 60.96 0)
 			(effects
@@
 			)
 		)
+		(pin "ESP32_RF_RX" input
+			(at 137.16 57.15 0)
+			(effects
+				(font
+					(size 1.27 1.27)
+				)
+				(justify right)
+			)
+		)
+		(pin "ESP32_RF_TX" output
+			(at 137.16 53.34 0)
+			(effects
+				(font
+					(size 1.27 1.27)
+				)
+				(justify right)
+			)
+		)
