File: pcb/mcu.kicad_sch (KiCad schematic)
At the start: 9 parts, among them U2 ESP32-WROOM-32U

Commit message: Merging in work from FSAE repo from when I forgot this one existed
Connections:
- net I2C_CLK: now also U2.37 (IO23); no longer U2.31 (IO19)
- net I2C_SDA: now also U2.36 (IO22); no longer U2.30 (IO18)
- net I2S_BCLK: now also U2.9 (IO33); no longer U2.33 (IO21)
- net I2S_LRC: now also U2.8 (IO32); no longer U2.10 (IO25)
- net I2S_SDIN: now also U2.31 (IO19); no longer U2.8 (IO32)
- net I2S_SDOUT: now also U2.33 (IO21); no longer U2.9 (IO33)
- net PTT: no longer U2.36 (IO22)
- net WARNING: no longer U2.37 (IO23)
- net SD_DATA1 renamed MAIN_LOOP
- net SD_DATA2 renamed FAULT
- net SD_DATA3 renamed RADIO ON/OFF

Commit message: Quite a few changes
Connections:
- net RADIO_STATUS is gone; now on net WARNING: U2.7 (IO35)
- net CAR_HEARTBEAT: now also U2.14 (IO12); no longer U2.29 (IO5)
- net FAULT: now also U2.30 (IO18); no longer U2.14 (IO12)
- net MAIN_LOOP: now also U2.10 (IO25); no longer U2.26 (IO4)
- net PTT: now also U2.26 (IO4)
- net RF_RX renamed ESP32_RF_RX
- net RF_TX renamed ESP32_RF_TX
- new net IS_RADIO_RECIEVING: U2.29 (IO5)
Changed lines of the file:
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@@
+	(wire
+		(pts
+			(xy 151.13 106.68) (xy 205.74 106.68)
+		)
+		(stroke
+			(width 0)
+			(type default)
+		)
+	)
 	(wire
 		(pts
@@
 	(wire
 		(pts
+			(xy 165.1 45.72) (xy 165.1 41.91)
+		)
+		(stroke
+			(width 0)
+			(type default)
+		)
+	)
+	(wire
+		(pts
 			(xy 151.13 91.44) (xy 205.74 91.44)
 		)
@@
 	(wire
 		(pts
-			(xy 165.1 45.72) (xy 165.1 41.91)
-		)
-		(stroke
-			(width 0)
-			(type default)
-		)
-	)
-	(wire
-		(pts
 			(xy 93.98 93.98) (xy 111.76 93.98)
 		)
@@
 	(wire
 		(pts
+			(xy 151.13 119.38) (xy 205.74 119.38)
+		)
+		(stroke
+			(width 0)
+			(type default)
+		)
+	)
+	(wire
+		(pts
 			(xy 175.26 41.91) (xy 165.1 41.91)
 		)
@@
 		)
 	)
-	(hierarchical_label "RF_TX"
+	(hierarchical_label "ESP32_RF_TX"
 		(shape output)
 		(at 182.88 104.14 0)
@@
 		)
 	)
+	(hierarchical_label "IS_RADIO_RECIEVING"
+		(shape input)
+		(at 205.74 88.9 0)
+		(effects
+			(font
+				(size 1.27 1.27)
+			)
+			(justify left)
+		)
+	)
 	(hierarchical_label "I2C_SDA"
 		(shape bidirectional)
@@
 		)
 	)
-	(hierarchical_label "RADIO_STATUS"
-		(shape input)
-		(at 205.74 134.62 0)
-		(effects
-			(font
-				(size 1.27 1.27)
-			)
-			(justify left)
-		)
-	)
 	(hierarchical_label "ESP32_RX"
 		(shape input)
@@
 		)
 	)
+	(hierarchical_label "I2S_SDOUT"
+		(shape output)
+		(at 170.18 111.76 0)
+		(effects
+			(font
+				(size 1.27 1.27)
+			)
+			(justify left)
+		)
+	)
+	(hierarchical_label "CAN_TX"
+		(shape output)
+		(at 194.31 124.46 0)
+		(effects
+			(font
+				(size 1.27 1.27)
+			)
+			(justify left)
+		)
+	)
+	(hierarchical_label "WARNING"
+		(shape output)
+		(at 205.74 134.62 0)
+		(effects
+			(font
+				(size 1.27 1.27)
+			)
+			(justify left)
+		)
+	)
+	(hierarchical_label "SD_CLK"
+		(shape output)
+		(at 158.75 96.52 0)
+		(effects
+			(font
+				(size 1.27 1.27)
+			)
+			(justify left)
+		)
+	)
+	(hierarchical_label "I2S_SDIN"
+		(shape input)
+		(at 170.18 109.22 0)
+		(effects
+			(font
+				(size 1.27 1.27)
+			)
+			(justify left)
+		)
+	)
+	(hierarchical_label "CAR_HEARTBEAT"
+		(shape output)
+		(at 205.74 91.44 0)
+		(effects
+			(font
+				(size 1.27 1.27)
+			)
+			(justify left)
+		)
+	)
 	(hierarchical_label "MAIN_LOOP"
 		(shape output)
+		(at 205.74 119.38 0)
+		(effects
+			(font
+				(size 1.27 1.27)
+			)
+			(justify left)
+		)
+	)
+	(hierarchical_label "ESP32_RF_RX"
+		(shape input)
+		(at 182.88 101.6 0)
+		(effects
+			(font
+				(size 1.27 1.27)
+			)
+			(justify left)
+		)
+	)
+	(hierarchical_label "CAN_RX"
+		(shape input)
+		(at 194.31 121.92 0)
+		(effects
+			(font
+				(size 1.27 1.27)
+			)
+			(justify left)
+		)
+	)
+	(hierarchical_label "FAULT"
+		(shape output)
+		(at 205.74 106.68 0)
+		(effects
+			(font
+				(size 1.27 1.27)
+			)
+			(justify left)
+		)
+	)
+	(hierarchical_label "I2S_BCLK"
+		(shape output)
+		(at 170.18 129.54 0)
+		(effects
+			(font
+				(size 1.27 1.27)
+			)
+			(justify left)
+		)
+	)
+	(hierarchical_label "BOOT_SELECT"
+		(shape input)
+		(at 205.74 69.85 0)
+		(effects
+			(font
+				(size 1.27 1.27)
+			)
+			(justify left)
+		)
+	)
+	(hierarchical_label "PTT"
+		(shape output)
 		(at 205.74 86.36 0)
 		(effects
 			(font
-				(size 1.27 1.27)
-			)
-			(justify left)
-		)
-	)
-	(hierarchical_label "I2S_SDOUT"
-		(shape output)
-		(at 170.18 111.76 0)
-		(effects
-			(font
-				(size 1.27 1.27)
-			)
-			(justify left)
-		)
-	)
-	(hierarchical_label "CAN_TX"
-		(shape output)
-		(at 194.31 124.46 0)
-		(effects
-			(font
-				(size 1.27 1.27)
-			)
-			(justify left)
-		)
-	)
-	(hierarchical_label "SD_CLK"
-		(shape output)
-		(at 158.75 96.52 0)
-		(effects
-			(font
-				(size 1.27 1.27)
-			)
-			(justify left)
-		)
-	)
-	(hierarchical_label "WARNING"
-		(shape output)
-		(at 205.74 116.84 0)
-		(effects
-			(font
-				(size 1.27 1.27)
-			)
-			(justify left)
-		)
-	)
-	(hierarchical_label "I2S_SDIN"
-		(shape input)
-		(at 170.18 109.22 0)
-		(effects
-			(font
-				(size 1.27 1.27)
-			)
-			(justify left)
-		)
-	)
-	(hierarchical_label "RF_RX"
-		(shape input)
-		(at 182.88 101.6 0)
-		(effects
-			(font
-				(size 1.27 1.27)
-			)
-			(justify left)
-		)
-	)
-	(hierarchical_label "CAN_RX"
-		(shape input)
-		(at 194.31 121.92 0)
-		(effects
-			(font
-				(size 1.27 1.27)
-			)
-			(justify left)
-		)
-	)
-	(hierarchical_label "I2S_BCLK"
-		(shape output)
-		(at 170.18 129.54 0)
-		(effects
-			(font
-				(size 1.27 1.27)
-			)
-			(justify left)
-		)
-	)
-	(hierarchical_label "BOOT_SELECT"
-		(shape input)
-		(at 205.74 69.85 0)
-		(effects
-			(font
-				(size 1.27 1.27)
-			)
-			(justify left)
-		)
-	)
-	(hierarchical_label "CAR_HEARTBEAT"
-		(shape output)
-		(at 205.74 88.9 0)
-		(effects
-			(font
-				(size 1.27 1.27)
-			)
-			(justify left)
-		)
-	)
-	(hierarchical_label "FAULT"
-		(shape output)
-		(at 205.74 91.44 0)
-		(effects
-			(font
-				(size 1.27 1.27)
-			)
-			(justify left)
-		)
-	)
-	(hierarchical_label "PTT"
-		(shape output)
-		(at 205.74 114.3 0)
-		(effects
-			(font
